File: test.brd (EAGLE design)
At the start: 101.6 x 53.3 mm, 60 parts, among them IC2 ATMEGA1280-16AU, IC4 MC33269D-5.0, IC6 FT232RL, IC7 LM358D, Q2 16MHz, T1 NDT2955, X2 DC21MMX

Commit message: test output
Parts:
- moved IC2 13.4 mm to (50.8, 28.3)
- moved JP2 10.7 mm to (95.2, 19.1)
- moved JP1 10.7 mm to (95.2, 39.4)
- moved PWMH 10.4 mm to (33.0, 50.8)
- moved ADCH 10.4 mm to (82.5, 2.54)
- moved ADCL 10.4 mm to (59.7, 2.54)
- moved COMMUNICATION 10.4 mm to (77.5, 50.8)
- moved PWML 10.4 mm to (54.6, 50.8)
- moved X2 9.65 mm to (6.83, 4.93)
- moved X4 9.20 mm to (-0.74, 38.1)
- moved IC4 8.37 mm to (4.68, 17.8)
- moved POWER 7.90 mm to (39.4, 2.54)
- moved IC6 7.37 mm to (18.3, 39.1)
- moved T1 6.44 mm to (7.15, 27.4)
- moved Q2 6.26 mm to (43.2, 13.2)
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
Commit message: test output
Parts:
- moved X4 4.55 mm to (3.81, 38.1), turned to 270 degrees
- moved X2 3.77 mm to (5.33, 8.38), turned to 90 degrees
- moved IC4 2.30 mm to (6.99, 17.8), turned to 90 degrees
- turned T1 to 90 degrees
- turned C6 to 270 degrees
- turned C7 to 270 degrees
- turned D1 to 270 degrees
- turned IC7 to 270 degrees
- turned ICSP to 270 degrees
- turned JP1 to 90 degrees
- turned JP2 to 90 degrees
- turned Q2 to 90 degrees
- turned RESET-EN to 270 degrees
- turned X3 to 270 degrees
Changed lines of the file:
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@@
         <element name="C4" library="rcl" package="C0805RND" value="100n" x="26.416" y="44.196" smashed="yes"/>
         <element name="C5" library="rcl" package="C0805RND" value="100n" x="16.256" y="18.796" smashed="yes"/>
-        <element name="C6" library="rcl" package="SMC_D" value="100u" x="22.86" y="6.096" smashed="yes" rot="R90"/>
-        <element name="C7" library="rcl" package="SMC_D" value="100u" x="28.448" y="6.096" smashed="yes" rot="R90"/>
+        <element name="C6" library="rcl" package="SMC_D" value="100u" x="22.86" y="6.096" smashed="yes" rot="R270"/>
+        <element name="C7" library="rcl" package="SMC_D" value="100u" x="28.448" y="6.096" smashed="yes" rot="R270"/>
         <element name="C9" library="rcl" package="C0805RND" value="100n" x="64.389" y="37.465" smashed="yes" rot="R180"/>
         <element name="COMMUNICATION" library="pinhead" package="1X08" value="" x="77.47" y="50.8" locked="yes" smashed="yes" rot="R180">
           <attribute name="VALUE" x="87.63" y="53.975" size="1.27" layer="27" rot="R180"/>
         </element>
-        <element name="D1" library="diode" package="SMB" value="" x="17.272" y="9.144" smashed="yes" rot="R90">
+        <element name="D1" library="diode" package="SMB" value="" x="17.272" y="9.144" smashed="yes" rot="R270">
           <attribute name="VALUE" x="13.843" y="11.303" size="1.27" layer="27" rot="R270"/>
         </element>
         <element name="F1" library="rcl" package="L1812" value="500mA" x="18.288" y="30.48" smashed="yes"/>
         <element name="IC2" library="atmel-2005" package="TQFP100" value="ATMEGA1280-16AU" x="50.8" y="28.3464" smashed="yes"/>
-        <element name="IC4" library="linear" package="DPACK" value="MC33269D-5.0" x="4.685" y="17.78" smashed="yes" rot="R270"/>
+        <element name="IC4" library="linear" package="DPACK" value="MC33269D-5.0" x="6.985" y="17.78" smashed="yes" rot="R90"/>
         <element name="IC6" library="SmartPrj" package="SSOP28" value="FT232RL" x="18.288" y="39.116" smashed="yes"/>
-        <element name="IC7" library="linear" package="SO08" value="LM358D" x="18.796" y="22.606" smashed="yes" rot="R90"/>
-        <element name="ICSP" library="pinhead" package="2X03" value="ICSP" x="64.897" y="27.94" locked="yes" smashed="yes" rot="R90"/>
-        <element name="JP1" library="pinhead" package="2X08" value="" x="95.25" y="39.37" locked="yes" smashed="yes" rot="R270">
+        <element name="IC7" library="linear" package="SO08" value="LM358D" x="18.796" y="22.606" smashed="yes" rot="R270"/>
+        <element name="ICSP" library="pinhead" package="2X03" value="ICSP" x="64.897" y="27.94" locked="yes" smashed="yes" rot="R270"/>
+        <element name="JP1" library="pinhead" package="2X08" value="" x="95.25" y="39.37" locked="yes" smashed="yes" rot="R90">
           <attribute name="VALUE" x="99.695" y="29.21" size="1.27" layer="27" rot="R90"/>
         </element>
-        <element name="JP2" library="pinhead" package="2X08" value="" x="95.25" y="19.05" locked="yes" smashed="yes" rot="R270">
+        <element name="JP2" library="pinhead" package="2X08" value="" x="95.25" y="19.05" locked="yes" smashed="yes" rot="R90">
           <attribute name="VALUE" x="99.695" y="8.89" size="1.27" layer="27" rot="R90"/>
         </element>
@@
           <attribute name="VALUE" x="73.66" y="38.354" size="1.27" layer="27" rot="R270"/>
         </element>
-        <element name="Q2" library="crystal" package="HC49/S" value="16MHz" x="43.18" y="13.208" smashed="yes" rot="R270"/>
+        <element name="Q2" library="crystal" package="HC49/S" value="16MHz" x="43.18" y="13.208" smashed="yes" rot="R90"/>
         <element name="R10" library="rcl" package="R0805RND" value="10k" x="16.256" y="16.256" smashed="yes" rot="R180"/>
         <element name="R11" library="SmartPrj" package="RCL_0805RND" value="1K" x="26.416" y="26.416" smashed="yes"/>
@@
         <element name="R8" library="rcl" package="R0805RND" value="1K" x="80.772" y="34.544" smashed="yes" rot="R180"/>
         <element name="R9" library="rcl" package="R0805RND" value="1k" x="26.416" y="28.956" smashed="yes"/>
-        <element name="RESET-EN" library="jumper" package="SJ" value="" x="30.48" y="20.955" smashed="yes" rot="R90">
+        <element name="RESET-EN" library="jumper" package="SJ" value="" x="30.48" y="20.955" smashed="yes" rot="R270">
           <attribute name="VALUE" x="30.48" y="20.5549" size="0.02" layer="27" rot="R270"/>
         </element>
@@
           <attribute name="VALUE" x="77.216" y="33.02" size="1.27" layer="27" ratio="10" rot="R180"/>
         </element>
-        <element name="T1" library="zetex" package="SOT223" value="NDT2955" x="7.147" y="27.432" smashed="yes" rot="R270"/>
+        <element name="T1" library="zetex" package="SOT223" value="NDT2955" x="7.112" y="27.432" smashed="yes" rot="R90"/>
         <element name="TX" library="led" package="0805RND" value="" x="26.416" y="34.036" smashed="yes" rot="R180">
           <attribute name="VALUE" x="28.956" y="36.576" size="1.27" layer="27" rot="R180"/>
@@
         <element name="U$2" library="SmartPrj" package="FIDUCIA-MOUNT" value="FIDUCIALMOUNT" x="36.703" y="17.653" locked="yes" smashed="yes"/>
         <element name="U$3" library="SmartPrj" package="FIDUCIA-MOUNT" value="FIDUCIALMOUNT" x="19.812" y="50.8" smashed="yes"/>
-        <element name="X2" library="powersupply" package="DC-21MM" value="DC21MMX" x="6.8326" y="4.9276" locked="yes" smashed="yes" rot="R270"/>
-        <element name="X3" library="jumper" package="JP4" value="" x="31.75" y="33.274" locked="yes" smashed="yes" rot="R90">
+        <element name="X2" library="powersupply" package="DC-21MM" value="DC21MMX" x="5.334" y="8.382" locked="yes" smashed="yes" rot="R90"/>
+        <element name="X3" library="jumper" package="JP4" value="" x="31.75" y="33.274" locked="yes" smashed="yes" rot="R270">
           <attribute name="VALUE" x="27.686" y="38.354" size="1.27" layer="27" ratio="10" rot="R270"/>
         </element>
-        <element name="X4" library="SmartPrj" package="PN61729" value="" x="-0.74" y="38.1" locked="yes" smashed="yes" rot="R90">
+        <element name="X4" library="SmartPrj" package="PN61729" value="" x="3.81" y="38.1" locked="yes" smashed="yes" rot="R270">
           <attribute name="VALUE" x="-5.08" y="30.48" size="1.27" layer="27"/>
         </element>
